File: HV-terminal-branch-board_2-4/HV-terminal-branch-board-2-4.kicad_pcb (KiCad board)
At the start: 2 copper layers, 80 x 30 mm, 11 parts, among them J1 Conn_01x01_Female_M6_hole, J2 Conn_01x01_Female_M6_hole, J3 Conn_01x01_Female_M6_hole, J4 Conn_01x01_Female_M6_hole, J5 Conn_01x01_Female_M6_hole, J6 Conn_01x01_Female_M6_hole

Commit message: add 2-4
add 2-4
Connections:
- J1 pad 1: VBAT+ -> VBAT(+/-)
- J2 pad 1: VBAT- -> VBAT(+/-)
- J3 pad 1: VBAT+ -> VBAT(+/-)
- J4 pad 1: VBAT+ -> VBAT(+/-)
- J5 pad 1: VBAT- -> VBAT(+/-)
- J6 pad 1: VBAT- -> VBAT(+/-)
Routing:
- net VBAT(+/-): track 0.00 -> 61.3 mm, vias 0 -> 174
- net VBAT-: track 30.6 -> 0.00 mm, vias 82 -> 0
- net VBAT+: track 30.6 -> 0.00 mm, vias 81 -> 0
- added copper zone on B.Cu, net VBAT(+/-)
- added copper zone on F.Cu, net VBAT(+/-)
- removed copper zone on B.Cu, net VBAT+
- removed copper zone on F.Cu, net VBAT+
- removed copper zone on B.Cu, net VBAT-
- removed copper zone on F.Cu, net VBAT-
Other:
- board text added: "Allowable current: ~400A Assumption: track width 1A/mm 1oz -> 66mm * 2 both sides * 1oz = 132A 2oz -> 66mm * 2 both sides * 2oz = 264A 3oz -> 66mm * 2 both sides * 3oz = 396A <- this one!! 4oz -> 66mm * 2 both sides * 4oz = 528A 5oz -> 66mm * 2 both sides * 5oz = 660A 6oz -> 66mm * 2 both sides * 6oz = 792A 7oz -> 66mm * 2 both sides * 7oz = 924A 8oz -> 66mm * 2 both sides * 8oz = 1056A"
- board text added: "HV-branch-2-4 221021 V1.0"
- board text removed: "Allowable current: ~200A Assumption: track width 1A/mm 1oz -> 32mm * 2 both sides * 1oz = 64A 2oz -> 32mm * 2 both sides * 2oz = 128A 3oz -> 32mm * 2 both sides * 3oz = 196A <- this one!! 4oz -> 32mm * 2 both sides * 4oz = 256A 5oz -> 32mm * 2 both sides * 5oz = 320A 6oz -> 32mm * 2 both sides * 6oz = 384A 7oz -> 32mm * 2 both sides * 7oz = 448A 8oz -> 32mm * 2 both sides * 8oz = 512A"
- board text removed: "HV-branch-1-2 221021 V1.0"
