File: HV-terminal-branch-board_2-4/HV-terminal-branch-board-2-4.kicad_sch (KiCad schematic)
At the start: 11 parts, among them J1 Conn_01x01_Female_M6_hole, J2 Conn_01x01_Female_M6_hole, J3 Conn_01x01_Female_M6_hole, J4 Conn_01x01_Female_M6_hole, J5 Conn_01x01_Female_M6_hole, J6 Conn_01x01_Female_M6_hole

Commit message: add 2-4
add 2-4
Connections:
- net VBAT- is gone; now on net VBAT(+/-): J2.1 (Pin_1), J5.1 (Pin_1), J6.1 (Pin_1)
- net VBAT+ renamed VBAT(+/-)
Other:
- note added: "INPUT_VBAT(+/-)"
- note added: "OUTPUT_VBAT(+/-)_1"
- note added: "OUTPUT_VBAT(+/-)_2"
- note added: "OUTPUT_VBAT(+/-)_3"
- note added: "OUTPUt_VBAT(+/-)_4"
- note removed: "INPUT_VBAT+"
- note removed: "INPUT_VBAT-"
- note removed: "OUTPUT_VBAT+_1"
- note removed: "OUTPUT_VBAT+_2"
- note removed: "OUTPUT_VBAT-_1"
- note removed: "OUTPUt_VBAT-_2"
- company: (none) -> teTra Aviation Corp.
- title: (none) -> HV terminal branch 2-4
Changed lines of the file:
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@@
 (kicad_sch (version 20211123) (generator eeschema)
   (paper "A4")
-  (junction (at 112.395 84.455) (diameter 0) (color 0 0 0 0)
+  (title_block
+    (title "HV terminal branch 2-4")
+    (date "2022-10-21")
+    (rev "1.0")
+    (company "teTra Aviation Corp.")
   )
   (junction (at 112.395 71.12) (diameter 0) (color 0 0 0 0)
   )
   (junction (at 119.38 71.12) (diameter 0) (color 0 0 0 0)
+  )
+  (junction (at 119.38 76.2) (diameter 0) (color 0 0 0 0)
   )
   (junction (at 119.38 84.455) (diameter 0) (color 0 0 0 0)
@@
   )
   (wire (pts (xy 125.095 89.535) (xy 119.38 89.535))
+    (stroke (width 0) (type default) (color 0 0 0 0))
+  )
+  (wire (pts (xy 119.38 76.2) (xy 119.38 84.455))
     (stroke (width 0) (type default) (color 0 0 0 0))
   )
@@
     (stroke (width 0) (type default) (color 0 0 0 0))
   )
-  (wire (pts (xy 112.395 84.455) (xy 112.395 97.79))
-    (stroke (width 0) (type default) (color 0 0 0 0))
-  )
   (wire (pts (xy 106.68 71.12) (xy 112.395 71.12))
-    (stroke (width 0) (type default) (color 0 0 0 0))
-  )
-  (wire (pts (xy 106.68 84.455) (xy 112.395 84.455))
     (stroke (width 0) (type default) (color 0 0 0 0))
   )
@@
     (stroke (width 0) (type default) (color 0 0 0 0))
   )
-  (wire (pts (xy 112.395 84.455) (xy 119.38 84.455))
+  (wire (pts (xy 106.68 84.455) (xy 119.38 84.455))
     (stroke (width 0) (type default) (color 0 0 0 0))
   )
@@
     (stroke (width 0) (type default) (color 0 0 0 0))
   )
-  (text "INPUT_VBAT-" (at 88.265 78.74 0)
+  (text "INPUT_VBAT(+/-)" (at 88.265 78.74 0)
     (effects (font (size 1.27 1.27)) (justify left bottom))
   )
-  (text "OUTPUT_VBAT+_2" (at 139.065 76.2 0)
+  (text "OUTPUT_VBAT(+/-)_2" (at 139.065 76.2 0)
     (effects (font (size 1.27 1.27)) (justify left bottom))
   )
-  (text "INPUT_VBAT+" (at 88.265 64.77 0)
+  (text "INPUT_VBAT(+/-)" (at 88.265 64.77 0)
     (effects (font (size 1.27 1.27)) (justify left bottom))
   )
-  (text "OUTPUT_VBAT+_1" (at 139.065 71.12 0)
+  (text "OUTPUT_VBAT(+/-)_1" (at 139.065 71.12 0)
     (effects (font (size 1.27 1.27)) (justify left bottom))
   )
-  (text "OUTPUt_VBAT-_2" (at 139.065 88.9 0)
+  (text "OUTPUt_VBAT(+/-)_4" (at 139.065 88.9 0)
     (effects (font (size 1.27 1.27)) (justify left bottom))
   )
-  (text "OUTPUT_VBAT-_1" (at 139.065 84.455 0)
+  (text "OUTPUT_VBAT(+/-)_3" (at 139.065 84.455 0)
     (effects (font (size 1.27 1.27)) (justify left bottom))
   )
-  (global_label "VBAT+" (shape input) (at 112.395 60.96 90) (fields_autoplaced)
+  (global_label "VBAT(+{slash}-)" (shape input) (at 112.395 60.96 90) (fields_autoplaced)
     (effects (font (size 1.27 1.27)) (justify left))
-    (property "Intersheet References" "${INTERSHEET_REFS}" (id 0) (at 112.3156 52.5598 90)
+    (property "Intersheet References" "${INTERSHEET_REFS}" (id 0) (at 112.3156 47.9636 90)
       (effects (font (size 1.27 1.27)) (justify left) hide)
     )
   )
-  (global_label "VBAT-" (shape input) (at 112.395 97.79 270) (fields_autoplaced)
-    (effects (font (size 1.27 1.27)) (justify right))
-    (property "Intersheet References" "${INTERSHEET_REFS}" (id 0) (at 112.3156 106.1902 90)
-      (effects (font (size 1.27 1.27)) (justify right) hide)
-    )
-  )
